File: Hardware/Prototipo_MCEE/Prototipo_MCEE.kicad_sch (KiCad schematic)
At the start: 0 parts

Commit message: bluepill
Parts:
- added C10, C11, C3, C4: 104u, Capacitor_SMD:C_0201_0603Metric, symbol Device:C
- added C13, C14, C15, C16: 20p, Capacitor_SMD:C_0201_0603Metric, symbol Device:C
- added J3, J4: Header_20, symbol Connector_Generic:Conn_01x20
- added R6: 1M, Resistor_SMD:R_0201_0603Metric, symbol Device:R
- added U1: STM32F103C8Tx, Package_QFP:LQFP-48_7x7mm_P0.5mm, symbol MCU_ST_STM32F1:STM32F103C8Tx
- added Y2: 8MHz, Crystal:Resonator-2Pin_W10.0mm_H5.0mm, symbol Device:Crystal
- added Y3: 32768KHz, Crystal:Resonator-2Pin_W10.0mm_H5.0mm, symbol Device:Crystal
Connections:
- new net: C13.1, C14.1
- new net: U1.35 (VSS_2), U1.47 (VSS)
- new net +3V3: C10.1, C11.1, C3.1, C4.1
- new net 5v: J4.3 (Pin_3)
- new net BOOT0: U1.44 (BOOT0)
- new net BOOT1: U1.20 (PB2/BOOT1)
- new net GND: C10.2, C11.2, C15.1, C16.1, C3.2, C4.2, J3.19 (Pin_19), J3.20 (Pin_20), J4.2 (Pin_2), U1.23 (VSS_1), U1.35 (VSS_2), U1.47 (VSS), U1.8 (VSSA)
- new net NRST: J3.17 (Pin_17)
- new net OSCIN: C13.2, R6.1, U1.5 (OSCIN), Y2.2
- new net OSCOUT: C14.2, R6.2, U1.6 (OSCOUT), Y2.1
- new net PA0: J3.5 (Pin_5), U1.10 (PA0)
- new net PA1: J3.6 (Pin_6), U1.11 (PA1)
- new net PA10: J4.14 (Pin_14), U1.31 (PA10)
- new net PA11: J4.13 (Pin_13), U1.32 (PA11)
- new net PA12: J4.12 (Pin_12), U1.33 (PA12)
- new net PA15: J4.11 (Pin_11), U1.38 (PA15)
- new net PA2: J3.7 (Pin_7), U1.12 (PA2)
- new net PA3: J3.8 (Pin_8), U1.13 (PA3)
- new net PA4: J3.9 (Pin_9), U1.14 (PA4)
- new net PA5: J3.10 (Pin_10), U1.15 (PA5)
- new net PA6: J3.11 (Pin_11), U1.16 (PA6)
- new net PA7: J3.12 (Pin_12), U1.17 (PA7)
- new net PA8: J4.16 (Pin_16), U1.29 (PA8)
- new net PA9: J4.15 (Pin_15), U1.30 (PA9)
- new net PB0: J3.13 (Pin_13), U1.18 (PB0)
- new net PB1: J3.14 (Pin_14), U1.19 (PB1)
- new net PB10: J3.15 (Pin_15), U1.21 (PB10)
- new net PB11: J3.16 (Pin_16), U1.22 (PB11)
- new net PB12: J4.20 (Pin_20), U1.25 (PB12)
- new net PB13: J4.19 (Pin_19), U1.26 (PB13)
- new net PB14: J4.18 (Pin_18), U1.27 (PB14)
- new net PB15: J4.17 (Pin_17), U1.28 (PB15)
- new net PB3: J4.10 (Pin_10), U1.39 (PB3)
- new net PB4: J4.9 (Pin_9), U1.40 (PB4)
- new net PB5: J4.8 (Pin_8), U1.41 (PB5)
- new net PB6: J4.7 (Pin_7), U1.42 (PB6)
- new net PB7: J4.6 (Pin_6), U1.43 (PB7)
- new net PB8: J4.5 (Pin_5), U1.45 (PB8)
- new net PB9: J4.4 (Pin_4), U1.46 (PB9)
- new net PC13: J3.2 (Pin_2), U1.2 (PC13)
- new net PC14: C15.2, J3.3 (Pin_3), U1.3 (PC14), Y3.2
- new net PC15: C16.2, J3.4 (Pin_4), U1.4 (PC15), Y3.1
- new net RESET: U1.7 (NRST)
- new net SWCLK: U1.37 (SWCLK)
- new net SWIO: U1.34 (SWIO)
- new net VBAT: J3.1 (Pin_1), U1.1 (VBAT)
- new net VCC3V3: J3.18 (Pin_18), J4.1 (Pin_1), U1.24 (VDD_1), U1.36 (VDD_2), U1.48 (VDD_3), U1.9 (VDDA)
