File: Hardware/PROTOTIPO_V9/Prototipo/Modulo RTC.kicad_sch (KiCad schematic)
At the start: 0 parts

Commit message: Esquematico RTC
Parts:
- added U6: 3013, 3013:MODULE_3013, symbol 3013:3013
Connections:
- new net: U6.SH1 (SHIELD), U6.SH2 (SHIELD)
- new net +3V3: U6.1 (3.3V)
- new net GND: U6.2 (GND)
- new net RTC_SCL: U6.3 (SCL)
- new net RTC_SDA: U6.4 (SDA)

Commit message: Bus de salida
Connections:
- no-connect marks 0 -> 6
Changed lines of the file:
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@@
 	(generator_version "9.0")
 	(paper "A4")
+	(no_connect
+		(at 161.29 85.09)
+	)
+	(no_connect
+		(at 130.81 100.33)
+	)
+	(no_connect
+		(at 130.81 87.63)
+	)
+	(no_connect
+		(at 161.29 92.71)
+	)
+	(no_connect
+		(at 161.29 95.25)
+	)
+	(no_connect
+		(at 132.08 90.17)
+	)
 	(wire
 		(pts

Commit message: sch ILI9341
Connections:
- no-connect marks 6 -> 5
Changed lines of the file:
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@@
 		(at 161.29 95.25)
-	)
-	(no_connect
-		(at 132.08 90.17)
 	)
 	(wire

Commit message: Asignación de huellas
Parts:
- U6: footprint 3013:MODULE_3013 -> footprints_proyecto:MODULE_3013
Changed lines of the file:
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@@
 			)
 		)
-		(property "Footprint" "3013:MODULE_3013"
+		(property "Footprint" "footprints_proyecto:MODULE_3013"
 			(at 146.05 92.71 0)
 			(effects
