File: Hardware/PROTOTIPO_V9/Prototipo/Modulo ADC.kicad_sch (KiCad schematic)
At the start: 0 parts

Commit message: sch ILI9341 y sch ADS1115
Parts:
- added R13: 10k, symbol Device:R_Small_US
- added U10: ADS1115IDGS, Package_SO:TSSOP-10_3x3mm_P0.5mm, symbol Analog_ADC:ADS1115IDGS
Connections:
- new net +5V: R13.1, U10.8 (VDD)
- new net ADC_IN0: U10.4 (AIN0)
- new net ADC_SCL: U10.10 (SCL)
- new net ADC_SDA: R13.2, U10.9 (SDA)
- new net GND: U10.1 (ADDR), U10.3 (GND)
- no-connect marks 0 -> 4

Commit message: sch ILI9341
Connections:
- net ADC_IN2: now reaches U10.6 (AIN2)
- net ADC_IN3: now reaches U10.7 (AIN3)
- no-connect marks 4 -> 2
Changed lines of the file:
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@@
-	)
-	(no_connect
-		(at 139.7 95.25)
 	)
 	(no_connect
@@
 		(at 160.02 87.63)
 	)
-	(no_connect
-		(at 139.7 97.79)
+	(wire
+		(pts
+			(xy 134.62 97.79) (xy 139.7 97.79)
+		)
+		(stroke
+			(width 0)
+			(type default)
+		)
 	)
 	(wire
@@
 		(pts
 			(xy 168.91 88.9) (xy 168.91 95.25)
+		)
+		(stroke
+			(width 0)
+			(type default)
+		)
+	)
+	(wire
+		(pts
+			(xy 134.62 95.25) (xy 139.7 95.25)
 		)
 		(stroke
@@
 		)
 	)
+	(hierarchical_label "ADC_IN3"
+		(shape input)
+		(at 134.62 97.79 180)
+		(effects
+			(font
+				(size 1.27 1.27)
+			)
+			(justify right)
+		)
+	)
 	(hierarchical_label "ADC_IN0"
 		(shape input)
@@
 		(effects
 			(font
+				(size 1.27 1.27)
+			)
+			(justify right)
+		)
+	)
+	(hierarchical_label "ADC_IN2"
+		(shape input)
+		(at 134.62 95.25 180)
+		(effects
+			(font

Commit message: Asignación de huellas
Parts:
- R13: footprint (none) -> Resistor_THT:R_Axial_DIN0207_L6.3mm_D2.5mm_P10.16mm_Horizontal
Changed lines of the file:
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@@
 			)
 		)
-		(property "Footprint" ""
+		(property "Footprint" "Resistor_THT:R_Axial_DIN0207_L6.3mm_D2.5mm_P10.16mm_Horizontal"
 			(at 168.91 86.36 0)
 			(effects

Commit message: Esquematico TR de Corriente
Connections:
- net ADC_IN1: now reaches U10.5 (AIN1)
- no-connect marks 2 -> 1
Changed lines of the file:
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@@
-	)
-	(no_connect
-		(at 139.7 92.71)
 	)
 	(no_connect
@@
 	(wire
 		(pts
+			(xy 134.62 92.71) (xy 139.7 92.71)
+		)
+		(stroke
+			(width 0)
+			(type default)
+		)
+	)
+	(wire
+		(pts
 			(xy 149.86 74.93) (xy 149.86 80.01)
 		)
@@
 			)
 			(justify left)
+		)
+	)
+	(hierarchical_label "ADC_IN1"
+		(shape input)
+		(at 134.62 92.71 180)
+		(effects
+			(font
+				(size 1.27 1.27)
+			)
+			(justify right)
 		)
 	)
@@
 		)
 		(instances
-			(project ""
+			(project "Prototipo"
 				(path "/f7e5c6e4-37d6-479e-ad19-5d06867b62e9/e27cf666-8cbc-4822-abe7-5197a8083313"
 					(reference "U10")
@@
 		)
 		(instances
-			(project ""
+			(project "Prototipo"
 				(path "/f7e5c6e4-37d6-479e-ad19-5d06867b62e9/e27cf666-8cbc-4822-abe7-5197a8083313"
 					(reference "R13")

Commit message: fp definitivos - Planteo de PCB con componentes
Parts:
- U10: footprint Package_SO:TSSOP-10_3x3mm_P0.5mm -> footprints_proyecto:MODULE_ADS1115
Changed lines of the file:
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@@
 			)
 		)
-		(property "Footprint" "Package_SO:TSSOP-10_3x3mm_P0.5mm"
+		(property "Footprint" "footprints_proyecto:MODULE_ADS1115"
 			(at 149.86 105.41 0)
 			(effects

Commit message: Migración de sch a BlackPill
Connections:
- net +5V renamed +3V3
Changed lines of the file:
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@@
 		)
 	)
-	(global_label "+5V"
+	(global_label "+3V3"
 		(shape input)
 		(at 149.86 72.39 90)
@@
 		)
 		(property "Intersheetrefs" "${INTERSHEET_REFS}"
-			(at 149.86 65.5343 90)
+			(at 149.86 64.3248 90)
 			(effects
 				(font
