File: Hardware/PROTOTIPO_V9/Prototipo/Modulo Sensor de V_A.kicad_sch (KiCad schematic)
At the start: 5 parts, among them J1 Screw_Terminal_01x02, U2 zmpt101b

Commit message: Migración de sch a BlackPill
Connections:
- net +5V renamed +3V3
Changed lines of the file:
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@@
 		)
 	)
-	(global_label "+5V"
+	(global_label "+3V3"
 		(shape input)
 		(at 200.66 88.9 0)
@@
 		)
 		(property "Intersheetrefs" "${INTERSHEET_REFS}"
-			(at 207.5157 88.9 0)
+			(at 208.7252 88.9 0)
 			(effects
 				(font
@@
 		)
 	)
-	(global_label "+5V"
+	(global_label "+3V3"
 		(shape input)
 		(at 173.99 57.15 180)
@@
 		)
 		(property "Intersheetrefs" "${INTERSHEET_REFS}"
-			(at 167.1343 57.15 0)
+			(at 165.9248 57.15 0)
 			(effects
 				(font
