File: Hardware/PROTOTIPO_V9/Prototipo/Modulo Ethernet.kicad_sch (KiCad schematic)
At the start: 0 parts

Commit message: Se agrega sch/fp W5500, ILI9341 y fp BluePill
Parts:
- added U8: W5500_ETHERNET_SHIELD, W5500_ETHERNET_SHIELD:W5500_ETHERNET_SHIELD, symbol W5500_ETHERNET_SHIELD:W5500_ETHERNET_SHIELD
Connections:
- new net +5V: U8.5V, U8.VIN
- new net CS_Eth: U8.D10
- new net CS_SD: U8.D4
- new net GND: U8.GND, U8.GND0, U8.GND1
- new net MISO: U8.D12
- new net MOSI: U8.D11
- new net RST_Eth: U8.RSTN (RSIN)
- no-connect marks 0 -> 28

Commit message: sch ILI9341
Connections:
- net CS_Eth renamed Eth_CS
- net CS_SD renamed SD_CS
- net RST_Eth renamed Eth_RST
Changed lines of the file:
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@@
-		)
-	)
-	(global_label "CS_SD"
-		(shape input)
-		(at 168.91 111.76 0)
-		(fields_autoplaced yes)
-		(effects
-			(font
-				(size 1.27 1.27)
-			)
-			(justify left)
-		)
-		(property "Intersheetrefs" "${INTERSHEET_REFS}"
-			(at 177.8218 111.76 0)
-			(effects
-				(font
-					(size 1.27 1.27)
-				)
-				(justify left)
-				(hide yes)
-			)
 		)
 	)
@@
 		(property "Intersheetrefs" "${INTERSHEET_REFS}"
 			(at 175.7657 83.82 0)
-			(effects
-				(font
-					(size 1.27 1.27)
-				)
-				(justify left)
-				(hide yes)
-			)
-		)
-	)
-	(global_label "RST_Eth"
-		(shape input)
-		(at 115.57 91.44 180)
-		(fields_autoplaced yes)
-		(effects
-			(font
-				(size 1.27 1.27)
-			)
-			(justify right)
-		)
-		(property "Intersheetrefs" "${INTERSHEET_REFS}"
-			(at 105.1464 91.44 0)
-			(effects
-				(font
-					(size 1.27 1.27)
-				)
-				(justify right)
-				(hide yes)
-			)
-		)
-	)
-	(global_label "CS_Eth"
-		(shape input)
-		(at 168.91 93.98 0)
-		(fields_autoplaced yes)
-		(effects
-			(font
-				(size 1.27 1.27)
-			)
-			(justify left)
-		)
-		(property "Intersheetrefs" "${INTERSHEET_REFS}"
-			(at 178.366 93.98 0)
 			(effects
 				(font
@@
 		)
 	)
+	(hierarchical_label "SD_CS"
+		(shape input)
+		(at 168.91 111.76 0)
+		(effects
+			(font
+				(size 1.27 1.27)
+			)
+			(justify left)
+		)
+	)
+	(hierarchical_label "Eth_RST"
+		(shape input)
+		(at 115.57 91.44 180)
+		(effects
+			(font
+				(size 1.27 1.27)
+			)
+			(justify right)
+		)
+	)
+	(hierarchical_label "Eth_CS"
+		(shape input)
+		(at 168.91 93.98 0)
+		(effects
+			(font
+				(size 1.27 1.27)
+			)
+			(justify left)
+		)
+	)

Commit message: ERC: 0 errores
Connections:
- net +5V: now also U8.5 (5V), U8.8 (VIN); no longer U8.5V, U8.VIN
- net Eth_CS: now also U8.31 (D10); no longer U8.D10
- net Eth_RST: now also U8.3 (RSIN); no longer U8.RSTN (RSIN)
- net GND: now also U8.35 (GND0), U8.6 (GND1), U8.7 (GND); no longer U8.GND, U8.GND0, U8.GND1
- net MISO: now also U8.33 (D12); no longer U8.D12
- net MOSI: now also U8.32 (D11); no longer U8.D11
- net SD_CS: now also U8.25 (D4); no longer U8.D4
Changed lines of the file:
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@@
 			)
 		)
-		(pin "D5"
+		(pin "13"
 		)
-		(pin "GND"
+		(pin "5"
 		)
-		(pin "D10"
+		(pin "35"
 		)
-		(pin "D0"
+		(pin "38"
 		)
-		(pin "D8"
+		(pin "12"
 		)
-		(pin "5V"
+		(pin "36"
 		)
-		(pin "D2"
+		(pin "14"
 		)
-		(pin "D1"
+		(pin "7"
 		)
-		(pin "GND1"
+		(pin "1"
 		)
-		(pin "5V"
+		(pin "4"
 		)
-		(pin "SCL"
+		(pin "6"
 		)
-		(pin "IOREF"
+		(pin "10"
 		)
-		(pin "A0"
+		(pin "9"
 		)
-		(pin "D13"
+		(pin "37"
 		)
-		(pin "AREF"
+		(pin "32"
 		)
-		(pin "A4"
+		(pin "34"
 		)
-		(pin "A5"
+		(pin "31"
 		)
-		(pin "D9"
+		(pin "11"
 		)
-		(pin "D6"
+		(pin "8"
 		)
-		(pin "D4"
+		(pin "30"
 		)
-		(pin "D3"
+		(pin "3"
 		)
-		(pin "GND"
+		(pin "2"
 		)
-		(pin "D11"
+		(pin "33"
 		)
-		(pin "A3"
+		(pin "29"
 		)
-		(pin "D7"
+		(pin "28"
 		)
-		(pin "D15"
+		(pin "27"
 		)
-		(pin "D14"
+		(pin "26"
 		)
-		(pin "A2"
+		(pin "25"
 		)
-		(pin "RSTN"
+		(pin "24"
 		)
-		(pin "GND0"
+		(pin "22"
 		)
-		(pin "RST"
+		(pin "21"
 		)
-		(pin "3.3V"
+		(pin "15"
 		)
-		(pin "NC"
+		(pin "16"
 		)
-		(pin "VIN"
+		(pin "17"
 		)
-		(pin "D12"
+		(pin "18"
 		)
-		(pin "MISO"
+		(pin "23"
 		)
-		(pin "A1"
+		(pin "20"
 		)
-		(pin "MOSI"
+		(pin "19"
 		)
 		(instances

Commit message: Asignación de huellas
Parts:
- U8: footprint W5500_ETHERNET_SHIELD:W5500_ETHERNET_SHIELD -> footprints_proyecto:W5500_ETHERNET_SHIELD
Changed lines of the file:
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@@
 			)
 		)
-		(property "Footprint" "W5500_ETHERNET_SHIELD:W5500_ETHERNET_SHIELD"
+		(property "Footprint" "footprints_proyecto:W5500_ETHERNET_SHIELD"
 			(at 124.46 124.46 0)
 			(effects

Commit message: PCB Prototipo final
Connections:
- net MISO: now also U8.17 (MISO); no longer U8.33 (D12)
- net MOSI: now also U8.19 (MOSI); no longer U8.32 (D11)
- net SCK: now reaches U8.16 (SCL)
- no-connect marks 28 -> 27
Changed lines of the file:
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@@
+	)
+	(no_connect
+		(at 165.1 88.9)
 	)
 	(no_connect
@@
 	)
 	(no_connect
-		(at 146.05 129.54)
-	)
-	(no_connect
 		(at 165.1 116.84)
 	)
@@
 	)
 	(no_connect
-		(at 140.97 129.54)
+		(at 165.1 91.44)
 	)
 	(no_connect
 		(at 148.59 129.54)
 	)
-	(no_connect
-		(at 138.43 129.54)
-	)
 	(wire
 		(pts
@@
 	(wire
 		(pts
-			(xy 165.1 88.9) (xy 168.91 88.9)
-		)
-		(stroke
-			(width 0)
-			(type default)
-		)
-	)
-	(wire
-		(pts
 			(xy 119.38 104.14) (xy 116.84 104.14)
 		)
@@
 	(wire
 		(pts
-			(xy 165.1 91.44) (xy 168.91 91.44)
-		)
-		(stroke
-			(width 0)
-			(type default)
-		)
-	)
-	(wire
-		(pts
 			(xy 165.1 83.82) (xy 168.91 83.82)
 		)
@@
 		)
 	)
+	(global_label "SCK"
+		(shape input)
+		(at 138.43 129.54 270)
+		(fields_autoplaced yes)
+		(effects
+			(font
+				(size 1.27 1.27)
+			)
+			(justify right)
+		)
+		(property "Intersheetrefs" "${INTERSHEET_REFS}"
+			(at 138.43 136.2747 90)
+			(effects
+				(font
+					(size 1.27 1.27)
+				)
+				(justify right)
+				(hide yes)
+			)
+		)
+	)
 	(global_label "+5V"
 		(shape input)
@@
 	(global_label "MISO"
 		(shape input)
-		(at 168.91 88.9 0)
-		(fields_autoplaced yes)
-		(effects
-			(font
-				(size 1.27 1.27)
-			)
-			(justify left)
-		)
-		(property "Intersheetrefs" "${INTERSHEET_REFS}"
-			(at 176.4914 88.9 0)
-			(effects
-				(font
-					(size 1.27 1.27)
-				)
-				(justify left)
+		(at 140.97 129.54 270)
+		(fields_autoplaced yes)
+		(effects
+			(font
+				(size 1.27 1.27)
+			)
+			(justify right)
+		)
+		(property "Intersheetrefs" "${INTERSHEET_REFS}"
+			(at 140.97 137.1214 90)
+			(effects
+				(font
+					(size 1.27 1.27)
+				)
+				(justify right)
 				(hide yes)
 			)
@@
 	(global_label "MOSI"
 		(shape input)
-		(at 168.91 91.44 0)
-		(fields_autoplaced yes)
-		(effects
-			(font
-				(size 1.27 1.27)
-			)
-			(justify left)
-		)
-		(property "Intersheetrefs" "${INTERSHEET_REFS}"
-			(at 176.4914 91.44 0)
-			(effects
-				(font
-					(size 1.27 1.27)
-				)
-				(justify left)
-				(hide yes)
-			)
+		(at 146.05 129.54 270)
+		(fields_autoplaced yes)
+		(effects
+			(font
+				(size 1.27 1.27)
+			)
+			(justify right)
+		)
+		(property "Intersheetrefs" "${INTERSHEET_REFS}"
+			(at 146.05 137.1214 90)
+			(effects
+				(font
+					(size 1.27 1.27)
+				)
+				(justify right)
+				(hide yes)
+			)
