File: Hardware/PROTOTIPO_V9/Prototipo/Prototipo.kicad_pcb (KiCad board)
At the start: 2 copper layers, 205.7 x 210.8 mm, 28 parts, among them J1 Screw_Terminal_01x02, J4 Conn_02x06_Counter_Clockwise, J5 Conn_02x06_Counter_Clockwise, J6 Conn_01x01, J7 Conn_01x01, J8 Conn_01x01, U10 ADS1115IDGS, U2 zmpt101b, U3 YAAJ_BlackPill_Part_Like_SWD_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, U5 LD1117V33, U6 3013, U7 KY-040, U8 W5500_ETHERNET_SHIELD, U9 CR2013-MI2120

Commit message: PCB Prototipo final
Parts:
- moved R1 101.5 mm to (147.3, 233.7), turned to -90 degrees
- moved U9 97.7 mm to (168.9, 243.8), turned to 90 degrees
- moved J4 65.9 mm to (218.4, 215.9), turned to -90 degrees
- moved U7 41.6 mm to (213.1, 190.6), turned to 0 degrees
- moved C1 7.62 mm to (281.9, 104.1)
- moved C2 7.62 mm to (281.9, 124.5)
- moved C3 7.62 mm to (213.4, 81.3)
- moved J5 7.62 mm to (160.0, 71.1)
- moved J8 7.62 mm to (218.4, 58.4)
- moved JP1 7.62 mm to (226.1, 127.0)
- moved JP2 7.62 mm to (223.5, 127.0)
- moved JP3 7.62 mm to (241.3, 127.0)
- moved JP4 7.62 mm to (238.8, 127.0)
- moved PS1 7.62 mm to (272.7, 55.9)
- moved R2 7.62 mm to (223.5, 63.5)
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Connections:
- U8 pad 16: unconnected-(U8-SCL-Pad16) -> SCK
- U8 pad 17: unconnected-(U8-MISO-Pad17) -> MISO
- U8 pad 19: unconnected-(U8-MOSI-Pad19) -> MOSI
- U8 pad 32: MOSI -> unconnected-(U8-D11-Pad32)
- U8 pad 33: MISO -> unconnected-(U8-D12-Pad33)
Routing:
- net SCK: track 35.6 -> 132.1 mm, vias 2 -> 6
- net /PCB2CONNECTION/LCD_MISO: track 119.4 -> 50.8 mm
- net MOSI: track 69.0 -> 137.2 mm, vias 2 -> 4
- net /PCB2CONNECTION/LCD_SCK: track 116.8 -> 53.3 mm
- net MISO: track 63.9 -> 127.0 mm, vias 2 -> 4
- net /PCB2CONNECTION/LCD_MOSI: track 111.8 -> 53.3 mm
- net /PCB2CONNECTION/LCD_DC: track 106.7 -> 53.3 mm
- net /PCB2CONNECTION/LCD_RST: track 106.7 -> 58.4 mm
- net /PCB2CONNECTION/LCD_CS: track 111.8 -> 68.6 mm
- net Net-(U9-LED): track 10.2 -> 45.7 mm
- net /PCB2CONNECTION/GND_: track 116.8 -> 86.4 mm
- net GND: track 517.7 -> 497.1 mm
- net /DS3231/RTC_SCL: track 193.1 -> 175.3 mm, vias 4 -> 7
- net /PCB2CONNECTION/ENC_SW: track 28.1 -> 12.7 mm
- net /PCB2CONNECTION/ENC_DT: track 28.1 -> 12.7 mm
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Other:
- board size 205.7 x 210.8 mm -> 205.7 x 213.4 mm
